File: hardware/mdb-interface.sch (KiCad schematic (older format))
At the start: 79 parts, among them IC1 ATMEGA644PA-A, J1 USB, K1 *, K2 *, P1 CONN_24, P10 CONN_1, P11 CONN_1, P12 CONN_1, P13 CONN_01X01, P2 CONN_12V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

Commit message: Leiterplattenbemaßung gesäubert, fixes #14
Parts:
- Q1, Q2: footprint (none) -> Transistors_SMD:sot23
Changed lines of the file:
@@
 F 0 "Q1" H 1650 3700 60  0000 R CNN
 F 1 "BCW67" H 1650 4000 60  0000 R CNN
-F 2 "" H 1650 3850 60  0000 C CNN
+F 2 "Transistors_SMD:sot23" H 1650 3850 60  0001 C CNN
 F 3 "" H 1650 3850 60  0000 C CNN
 	1    1650 3850
@@
 F 0 "Q2" H 2150 3900 60  0000 R CNN
 F 1 "BCW67" H 2150 4200 60  0000 R CNN
-F 2 "" H 2150 4050 60  0000 C CNN
+F 2 "Transistors_SMD:sot23" H 2150 4050 60  0001 C CNN
 F 3 "" H 2150 4050 60  0000 C CNN
 	1    2150 4050

Commit message: Platine angepasst, bereit zur Fertigungsvorbereitung, fixes #11
Parts:
- removed Q1, Q2: BCW67, Transistors_SMD:sot23, symbol PNP
- added Q1, Q2: BCW67, Transistors_SMD:sot23, symbol PNP_1B2E3C
- P13: footprint Connect:1pin -> Measurement_Points:Measurement_Point_Square-TH_Small
Connections:
- net +5V: now also Q1.2 (E)
- net MDB_MT: now also Q2.3 (C)
- net at R5.2: now also Q1.1 (B), Q2.2 (E)
- net at R1.2: now also Q1.3 (C), Q2.1 (B)
Changed lines of the file:
@@
 F 0 "P13" H 3800 9800 50  0000 C CNN
 F 1 "CONN_01X01" V 3900 9700 50  0000 C CNN
-F 2 "Connect:1pin" H 3800 9700 60  0001 C CNN
+F 2 "Measurement_Points:Measurement_Point_Square-TH_Small" H 3800 9700 60  0001 C CNN
 F 3 "" H 3800 9700 60  0000 C CNN
 	1    3800 9700
@@
 Connection ~ 1850 6050
 $Comp
-L PNP Q1
-U 1 1 54BBB005
+L PNP_1B2E3C Q1
+U 1 1 54BBDCA1
 P 1650 3850
 F 0 "Q1" H 1650 3700 60  0000 R CNN
@@
 $EndComp
 $Comp
-L PNP Q2
-U 1 1 54BBB1C4
+L PNP_1B2E3C Q2
+U 1 1 54BBE1C5
 P 2150 4050
 F 0 "Q2" H 2150 3900 60  0000 R CNN
