File: hardware/mdb-interface/mdb-interface.sch (KiCad schematic (older format))
At the start: 79 parts, among them IC1 ATMEGA644PA-A, J1 USB, K1 *, K2 *, P1 CONN_24, P10 CONN_1, P11 CONN_1, P12 CONN_1, P13 CONN_01X01, P2 CONN_12V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

Commit message: MDB Interface Platine: Änderungsnotiz zu 5V-Versorgung
Parts:
- C1, C10, C11, C12, C13, C14, C15, C4, C5, C6, C7, C8, C9: symbol C -> C-RESCUE-mdb-interface
- D1, D4, D6, D7, D8, D9: symbol LED -> LED-RESCUE-mdb-interface
- R1, R10, R11, R12, R13, R14, R15, R16, R17, R18, R19, R2, R3, R4, R5, R6, R7, R8, R9, ferrite1: symbol R -> R-RESCUE-mdb-interface
Other:
- note added: "TODO: Folgendes ist zur Zeit nur notdürftig manuell umgefrickelt, muss bei der nächsten Revision in Schaltplan und Layout rein.\nVCC nicht von VUSB, sondern von 12V\nüber 7805 beziehen. Vor dem 7805 eine Diode und einen Elko hinsetzen.\nAm 7805 eine Rückwärtsdiode 5V nach 12V, und Caps für Ein- und Ausgang."
Changed lines of the file:
@@
 EESchema Schematic File Version 2
+LIBS:mdb-interface-rescue
 LIBS:power
 LIBS:device
@@
 LIBS:memory
 LIBS:xilinx
-LIBS:special
 LIBS:microcontrollers
 LIBS:dsp
@@
 Connection ~ 6250 2850
 $Comp
-L R R8
+L R-RESCUE-mdb-interface R8
 U 1 1 531F7E15
 P 5750 2750
@@
 $EndComp
 $Comp
-L C C9
+L C-RESCUE-mdb-interface C9
 U 1 1 531F7DFE
 P 6050 2250
@@
 $EndComp
 $Comp
-L C C10
+L C-RESCUE-mdb-interface C10
 U 1 1 531F7DF3
 P 6250 3050
@@
 $EndComp
 $Comp
-L C C13
+L C-RESCUE-mdb-interface C13
 U 1 1 531CD1AD
 P 6950 1300
@@
 NoConn ~ 6000 8250
 $Comp
-L LED D7
+L LED-RESCUE-mdb-interface D7
 U 1 1 531C9351
 P 7050 8300
@@
 $EndComp
 $Comp
-L R R10
+L R-RESCUE-mdb-interface R10
 U 1 1 531C9350
 P 6600 8300
@@
 $EndComp
 $Comp
-L R R9
+L R-RESCUE-mdb-interface R9
 U 1 1 531C9334
 P 6550 7950
@@
 $EndComp
 $Comp
-L LED D6
+L LED-RESCUE-mdb-interface D6
 U 1 1 531C9333
 P 7000 7950
@@
 $EndComp
 $Comp
-L C C1
+L C-RESCUE-mdb-interface C1
 U 1 1 531B4437
 P 2250 7250
@@
 $EndComp
 $Comp
-L C C5
+L C-RESCUE-mdb-interface C5
 U 1 1 531B440A
 P 3850 6600
@@
 $EndComp
 $Comp
-L C C7
+L C-RESCUE-mdb-interface C7
 U 1 1 531B43E8
 P 4150 8550
@@
 $EndComp
 $Comp
-L LED D9
+L LED-RESCUE-mdb-interface D9
 U 1 1 531B41F0
 P 9900 3050
@@
 $EndComp
 $Comp
-L R R12
+L R-RESCUE-mdb-interface R12
 U 1 1 531B41EF
 P 10350 3050
@@
 $EndComp
 $Comp
-L C C14
+L C-RESCUE-mdb-interface C14
 U 1 1 531B4161
 P 6950 3350
@@
 $EndComp
 $Comp
-L C C15
+L C-RESCUE-mdb-interface C15
 U 1 1 531B3E2C
 P 8700 1450
@@
 BusRX
 $Comp
-L R R2
+L R-RESCUE-mdb-interface R2
 U 1 1 531B3D74
 P 1350 6050
@@
 $EndComp
 $Comp
-L LED D1
+L LED-RESCUE-mdb-interface D1
 U 1 1 531B3D44
 P 1600 5350
@@
 $EndComp
 $Comp
-L R R3
+L R-RESCUE-mdb-interface R3
 U 1 1 531B3D42
 P 1600 5800
@@
 $EndComp
 $Comp
-L R R7
+L R-RESCUE-mdb-interface R7
 U 1 1 531B3C8E
 P 2700 4900
@@
 $EndComp
 $Comp
-L LED D4
+L LED-RESCUE-mdb-interface D4
 U 1 1 531B3C88
 P 2700 4450
@@
 $EndComp
 $Comp
-L R R6
+L R-RESCUE-mdb-interface R6
 U 1 1 531B3C79
 P 2250 4900
@@
 BusTX
 $Comp
-L R R1
+L R-RESCUE-mdb-interface R1
 U 1 1 531B3BEC
 P 1150 4050
@@
 $EndComp
 $Comp
-L R R5
+L R-RESCUE-mdb-interface R5
 U 1 1 531B3BC9
 P 2250 3600
@@
 	6950 2250 6950 2350
 $Comp
-L R ferrite1
+L R-RESCUE-mdb-interface ferrite1
 U 1 1 53469E18
 P 8000 1400
@@
 $EndComp
 $Comp
-L C C12
+L C-RESCUE-mdb-interface C12
 U 1 1 5346AD75
 P 6700 1300
@@
 $EndComp
 $Comp
-L C C11
+L C-RESCUE-mdb-interface C11
 U 1 1 5346AD80
 P 6450 1300
@@
 PWM_5
 $Comp
-L LED D8
+L LED-RESCUE-mdb-interface D8
 U 1 1 5346C0F3
 P 9900 2750
@@
 $EndComp
 $Comp
-L R R11
+L R-RESCUE-mdb-interface R11
 U 1 1 5346C0FE
 P 10350 2750
@@
 $EndComp
 $Comp
-L R R13
+L R-RESCUE-mdb-interface R13
 U 1 1 5346ED73
 P 12300 4350
@@
 $EndComp
 $Comp
-L R R14
+L R-RESCUE-mdb-interface R14
 U 1 1 5346EF5E
 P 12300 5100
@@
 $EndComp
 $Comp
-L R R15
+L R-RESCUE-mdb-interface R15
 U 1 1 5346EF98
 P 12300 5800
@@
 $EndComp
 $Comp
-L R R16
+L R-RESCUE-mdb-interface R16
 U 1 1 5346EFB8
 P 14300 4350
@@
 $EndComp
 $Comp
-L R R17
+L R-RESCUE-mdb-interface R17
 U 1 1 5346EFD7
 P 14300 5100
@@
 $EndComp
 $Comp
-L R R18
+L R-RESCUE-mdb-interface R18
 U 1 1 5346EFF6
 P 14300 5800
@@
 $EndComp
 $Comp
-L C C4
+L C-RESCUE-mdb-interface C4
 U 1 1 5347010C
 P 2750 2800
@@
 +
 $Comp
-L R R19
+L R-RESCUE-mdb-interface R19
 U 1 1 53680430
 P 2300 7700
@@
 	8950 3250 9300 3250
 $Comp
-L C C6
+L C-RESCUE-mdb-interface C6
 U 1 1 53E257B2
 P 13450 7000
@@
 $EndComp
 $Comp
-L C C8
+L C-RESCUE-mdb-interface C8
 U 1 1 53E2582F
 P 13450 7450
@@
 Connection ~ 12950 7450
 $Comp
-L R R4
+L R-RESCUE-mdb-interface R4
 U 1 1 531B3D38
 P 1850 5800
@@
 	1    0    0    1
 $EndComp
+Text Notes 1850 5750 0    197  ~ 39
+TODO: Folgendes ist zur Zeit nur notdürftig manuell umgefrickelt, muss bei der nächsten Revision in Schaltplan und Layout rein.\nVCC nicht von VUSB, sondern von 12V\nüber 7805 beziehen. Vor dem 7805 eine Diode und einen Elko hinsetzen.\nAm 7805 eine Rückwärtsdiode 5V nach 12V, und Caps für Ein- und Ausgang.
 $EndSCHEMATC
